Commit message: update

File: urdf_description/urdf/urdf.xacro (robot description, xacro)
@@ -4,4 +4,6 @@
 <xacro:include filename="$(find urdf_description)/urdf/urdf.trans" />
 <xacro:include filename="$(find urdf_description)/urdf/urdf.gazebo" />
+<link name="base_footprint">
+  </link>
 <link name="base_link">
   <inertial>
@@ -104,4 +106,20 @@
   </collision>
 </link>
+<link name="laser">
+    <inertial>
+      <origin xyz="0 0 0" rpy="0 0 0"/>
+      <mass value="0.125"/>
+      <inertia ixx="0.000"  ixy="0"  ixz="0" iyy="0.000" iyz="0" izz="0.001" />
+    </inertial>
+</link>
+<joint name="lidar_joint" type="fixed">
+  <parent link="base_link"/>
+  <child link="laser"/>
+  <origin xyz="0 -0.03 0.15" rpy="0 0 1.57"/>
+</joint>
+<joint name="dummy_joint" type="fixed">
+  <parent link="base_footprint"/>
+  <child link="base_link"/>
+</joint>
 <joint name="Rev17" type="continuous">
   <origin xyz="0.0 -0.09904 -0.035" rpy="0 0 0"/>

Commit message: update

File: urdf_description/urdf/urdf.xacro (robot description, xacro)
@@ -5,4 +5,5 @@
 <xacro:include filename="$(find urdf_description)/urdf/urdf.gazebo" />
 <link name="base_footprint">
+  <origin xyz="0 0 0" rpy="0 0 0"/>
   </link>
 <link name="base_link">
@@ -116,9 +117,11 @@
   <parent link="base_link"/>
   <child link="laser"/>
-  <origin xyz="0 -0.03 0.15" rpy="0 0 1.57"/>
+  <!--origin xyz="0 -0.03 0.15" rpy="0 0 1.57"/-->
+  <origin xyz="0 0 0.1" rpy="0 0 1.57"/>
 </joint>
 <joint name="dummy_joint" type="fixed">
   <parent link="base_footprint"/>
   <child link="base_link"/>
+  <origin xyz="0 0 0.07" rpy="0 0 -1.57"/>
 </joint>
 <joint name="Rev17" type="continuous">

Commit message: up

File: urdf_description/urdf/urdf.xacro (robot description, xacro)
@@ -118,10 +118,10 @@
   <child link="laser"/>
   <!--origin xyz="0 -0.03 0.15" rpy="0 0 1.57"/-->
-  <origin xyz="0 0 0.1" rpy="0 0 1.57"/>
+  <origin xyz="0 0 0.1" rpy="0 0 0"/>
 </joint>
 <joint name="dummy_joint" type="fixed">
   <parent link="base_footprint"/>
   <child link="base_link"/>
-  <origin xyz="0 0 0.07" rpy="0 0 -1.57"/>
+  <origin xyz="0 0 0.07" rpy="0 0 0"/>
 </joint>
 <joint name="Rev17" type="continuous">

Commit message: go

File: urdf_description/urdf/urdf.xacro (robot description, xacro)
@@ -114,17 +114,18 @@
     </inertial>
 </link>
+<!--joint-->
 <joint name="lidar_joint" type="fixed">
   <parent link="base_link"/>
   <child link="laser"/>
   <!--origin xyz="0 -0.03 0.15" rpy="0 0 1.57"/-->
-  <origin xyz="0 0 0.1" rpy="0 0 0"/>
+  <origin xyz="0 0 0.1" rpy="0 0 1.57"/>
 </joint>
 <joint name="dummy_joint" type="fixed">
   <parent link="base_footprint"/>
   <child link="base_link"/>
-  <origin xyz="0 0 0.07" rpy="0 0 0"/>
+  <origin xyz="0 0 0.048" rpy="0 0 1.57"/>
 </joint>
 <joint name="Rev17" type="continuous">
-  <origin xyz="0.0 -0.09904 -0.035" rpy="0 0 0"/>
+  <origin xyz="0.0 -0.09904 -0.024" rpy="0 0 0"/>
   <parent link="base_link"/>
   <child link="wheel_2_1"/>
@@ -132,5 +133,5 @@
 </joint>
 <joint name="Rev18" type="continuous">
-  <origin xyz="-0.085771 0.04952 -0.035" rpy="0 0 0"/>
+  <origin xyz="-0.085771 0.04952 -0.024" rpy="0 0 0"/>
   <parent link="base_link"/>
   <child link="wheel_1_1"/>
@@ -138,5 +139,5 @@
 </joint>
 <joint name="Rev19" type="continuous">
-  <origin xyz="0.085771 0.04952 -0.035" rpy="0 0 0"/>
+  <origin xyz="0.085771 0.04952 -0.024" rpy="0 0 0"/>
   <parent link="base_link"/>
   <child link="wheel_3_1"/>

Commit message: update

File: urdf_description/urdf/urdf.xacro (robot description, xacro)
@@ -4,13 +4,13 @@
 <xacro:include filename="$(find urdf_description)/urdf/urdf.trans" />
 <xacro:include filename="$(find urdf_description)/urdf/urdf.gazebo" />
-<link name="base_footprint">
-  <origin xyz="0 0 0" rpy="0 0 0"/>
-  </link>
 <link name="base_link">
-  <inertial>
-    <origin xyz="0.0014632405775191286 0.008789062002822465 0.009289667535659163" rpy="0 0 0"/>
-    <mass value="3.5754408520918015"/>
-    <inertia ixx="0.006432" iyy="0.008693" izz="0.012797" ixy="0.000357" iyz="1.7e-05" ixz="-0.000138"/>
-  </inertial>
+  <!--inertial>
+    <!origin xyz="-0.0009504107610491734 -0.009453690875261649 0.06855931514078502" rpy="0 0 0"/>
+    <mass value="3.4980631377264046"/>
+    <inertia ixx="0.005992" iyy="0.008369" izz="0.01248" ixy="0.000384" iyz="4.7e-05" ixz="0.000156"/>
+    <origin xyz="0 0 0" rpy="0 0 0"/>
+    <mass value="0"/>
+    <inertia ixx="0" iyy="0" izz="0" ixy="0" iyz="0" ixz="0"/>
+  </inertial!-->
   <visual>
     <origin xyz="0 0 0" rpy="0 0 0"/>
@@ -27,65 +27,65 @@
   </collision>
 </link>
-<link name="wheel_2_1">
+<link name="wheel_link_1">
   <inertial>
-    <origin xyz="0.00010755761556894396 -0.008110733716275756 1.1541361448375032e-05" rpy="0 0 0"/>
-    <mass value="0.18489052459734032"/>
-    <inertia ixx="3.4e-05" iyy="5.4e-05" izz="3.4e-05" ixy="0.0" iyz="-0.0" ixz="-0.0"/>
+    <origin xyz="-9.278975567870437e-05 -0.007650950152439842 -2.8097213279051902e-05" rpy="0 0 0"/>
+    <mass value="0.17051038938064"/>
+    <inertia ixx="3.2e-05" iyy="5e-05" izz="3.2e-05" ixy="0.0" iyz="0.0" ixz="0.0"/>
   </inertial>
   <visual>
-    <origin xyz="-0.0 0.09904 0.035" rpy="0 0 0"/>
+    <origin xyz="-0.0 -0.11454 -0.02425" rpy="0 0 0"/>
     <geometry>
-      <mesh filename="package://urdf_description/meshes/wheel_2_1.stl" scale="0.001 0.001 0.001"/>
+      <mesh filename="package://urdf_description/meshes/wheel_link_1.stl" scale="0.001 0.001 0.001"/>
     </geometry>
     <material name="silver"/>
   </visual>
   <collision>
-    <origin xyz="-0.0 0.09904 0.035" rpy="0 0 0"/>
+    <origin xyz="-0.0 -0.11454 -0.02425" rpy="0 0 0"/>
     <geometry>
-      <mesh filename="package://urdf_description/meshes/wheel_2_1.stl" scale="0.001 0.001 0.001"/>
+      <mesh filename="package://urdf_description/meshes/wheel_link_1.stl" scale="0.001 0.001 0.001"/>
     </geometry>
   </collision>
 </link>
-<link name="wheel_1_1">
+<link name="wheel_link_2">
   <inertial>
-    <origin xyz="-0.00703002811317352 0.004045371745907196 -0.00010755761559414628" rpy="0 0 0"/>
-    <mass value="0.1848905245973405"/>
-    <inertia ixx="4.9e-05" iyy="3.9e-05" izz="3.4e-05" ixy="-8e-06" iyz="-0.0" ixz="-0.0"/>
+    <origin xyz="0.0066146071273707335 0.0038441124941529514 9.453176371182481e-05" rpy="0 0 0"/>
+    <mass value="0.17051038938064"/>
+    <inertia ixx="4.6e-05" iyy="3.6e-05" izz="3.2e-05" ixy="8e-06" iyz="0.0" ixz="0.0"/>
   </inertial>
   <visual>
-    <origin xyz="0.085771 -0.04952 0.035" rpy="0 0 0"/>
+    <origin xyz="0.099194 0.05727 -0.02425" rpy="0 0 0"/>
     <geometry>
-      <mesh filename="package://urdf_description/meshes/wheel_1_1.stl" scale="0.001 0.001 0.001"/>
+      <mesh filename="package://urdf_description/meshes/wheel_link_2.stl" scale="0.001 0.001 0.001"/>
     </geometry>
     <material name="silver"/>
   </visual>
   <collision>
-    <origin xyz="0.085771 -0.04952 0.035" rpy="0 0 0"/>
+    <origin xyz="0.099194 0.05727 -0.02425" rpy="0 0 0"/>
     <geometry>
-      <mesh filename="package://urdf_description/meshes/wheel_1_1.stl" scale="0.001 0.001 0.001"/>
+      <mesh filename="package://urdf_description/meshes/wheel_link_2.stl" scale="0.001 0.001 0.001"/>
     </geometry>
   </collision>
 </link>
-<link name="wheel_3_1">
+<link name="wheel_link_3">
   <inertial>
-    <origin xyz="0.007018486751699429 0.004065361970368803 -0.0001075576155941324" rpy="0 0 0"/>
-    <mass value="0.18489052459734032"/>
-    <inertia ixx="4.9e-05" iyy="3.9e-05" izz="3.4e-05" ixy="9e-06" iyz="0.0" ixz="0.0"/>
+    <origin xyz="-0.006606750578656451 0.003857720435697716 8.95155919554795e-05" rpy="0 0 0"/>
+    <mass value="0.17051038938064"/>
+    <inertia ixx="4.5e-05" iyy="3.7e-05" izz="3.2e-05" ixy="-8e-06" iyz="0.0" ixz="0.0"/>
   </inertial>
   <visual>
-    <origin xyz="-0.085771 -0.04952 0.035" rpy="0 0 0"/>
+    <origin xyz="-0.099194 0.05727 -0.02425" rpy="0 0 0"/>
     <geometry>
-      <mesh filename="package://urdf_description/meshes/wheel_3_1.stl" scale="0.001 0.001 0.001"/>
+      <mesh filename="package://urdf_description/meshes/wheel_link_3.stl" scale="0.001 0.001 0.001"/>
     </geometry>
     <material name="silver"/>
   </visual>
   <collision>
-    <origin xyz="-0.085771 -0.04952 0.035" rpy="0 0 0"/>
+    <origin xyz="-0.099194 0.05727 -0.02425" rpy="0 0 0"/>
     <geometry>
-      <mesh filename="package://urdf_description/meshes/wheel_3_1.stl" scale="0.001 0.001 0.001"/>
+      <mesh filename="package://urdf_description/meshes/wheel_link_3.stl" scale="0.001 0.001 0.001"/>
     </geometry>
   </collision>
 </link>
-<link name="lidar_1">
+<link name="lidar_link">
   <inertial>
     <origin xyz="-0.029581681955466045 0.042548549097526214 0.028542673476791153" rpy="0 0 0"/>
@@ -96,5 +96,5 @@
     <origin xyz="-0.029369 0.014322 -0.048" rpy="0 0 0"/>
     <geometry>
-      <mesh filename="package://urdf_description/meshes/lidar_1.stl" scale="0.001 0.001 0.001"/>
+      <mesh filename="package://urdf_description/meshes/lidar_link_1.stl" scale="0.001 0.001 0.001"/>
     </geometry>
     <material name="silver"/>
@@ -103,5 +103,5 @@
     <origin xyz="-0.029369 0.014322 -0.048" rpy="0 0 0"/>
     <geometry>
-      <mesh filename="package://urdf_description/meshes/lidar_1.stl" scale="0.001 0.001 0.001"/>
+      <mesh filename="package://urdf_description/meshes/lidar_link_1.stl" scale="0.001 0.001 0.001"/>
     </geometry>
   </collision>
@@ -121,31 +121,26 @@
   <origin xyz="0 0 0.1" rpy="0 0 1.57"/>
 </joint>
-<joint name="dummy_joint" type="fixed">
-  <parent link="base_footprint"/>
-  <child link="base_link"/>
-  <origin xyz="0 0 0.048" rpy="0 0 1.57"/>
-</joint>
-<joint name="Rev17" type="continuous">
-  <origin xyz="0.0 -0.09904 -0.024" rpy="0 0 0"/>
-  <parent link="base_link"/>
-  <child link="wheel_2_1"/>
-  <axis xyz="0.0 -1.0 -0.0"/>
-</joint>
-<joint name="Rev18" type="continuous">
-  <origin xyz="-0.085771 0.04952 -0.024" rpy="0 0 0"/>
-  <parent link="base_link"/>
-  <child link="wheel_1_1"/>
-  <axis xyz="0.866025 -0.5 0.0"/>
-</joint>
-<joint name="Rev19" type="continuous">
-  <origin xyz="0.085771 0.04952 -0.024" rpy="0 0 0"/>
-  <parent link="base_link"/>
-  <child link="wheel_3_1"/>
-  <axis xyz="0.866025 0.5 -0.0"/>
-</joint>
-<joint name="Rigid20" type="fixed">
+<joint name="Rigid1" type="fixed">
   <origin xyz="0.029369 -0.014322 0.048" rpy="0 0 0"/>
   <parent link="base_link"/>
-  <child link="lidar_1"/>
+  <child link="lidar_link"/>
+</joint>
+<joint name="Rev3" type="continuous">
+  <origin xyz="0.0 0.11454 0.02425" rpy="0 0 0"/>
+  <parent link="base_link"/>
+  <child link="wheel_link_1"/>
+  <axis xyz="0.0 1.0 -0.0"/>
+</joint>
+<joint name="Rev4" type="continuous">
+  <origin xyz="-0.099194 -0.05727 0.02425" rpy="0 0 0"/>
+  <parent link="base_link"/>
+  <child link="wheel_link_2"/>
+  <axis xyz="-0.866025 -0.5 -0.0"/>
+</joint>
+<joint name="Rev5" type="continuous">
+  <origin xyz="0.099194 -0.05727 0.02425" rpy="0 0 0"/>
+  <parent link="base_link"/>
+  <child link="wheel_link_3"/>
+  <axis xyz="0.866025 -0.5 -0.0"/>
 </joint>
 </robot>

Commit message: update

File: urdf_description/urdf/urdf.xacro (robot description, xacro)
@@ -126,4 +126,10 @@
   <child link="lidar_link"/>
 </joint>
+<joint name="Rigid2" type="fixed">
+  <origin xyz="0.029369 -0.014322 0.048" rpy="0 0 0"/>
+  <parent link="base_link"/>
+  <child link="lidar_1"/>
+</joint>
+<!--wheel joint-->
 <joint name="Rev3" type="continuous">
   <origin xyz="0.0 0.11454 0.02425" rpy="0 0 0"/>

Commit message: update

File: urdf_description/urdf/urdf.xacro (robot description, xacro)
@@ -114,5 +114,5 @@
     </inertial>
 </link>
-<!--joint-->
+<!--base-lidar joint-->
 <joint name="lidar_joint" type="fixed">
   <parent link="base_link"/>
@@ -121,15 +121,11 @@
   <origin xyz="0 0 0.1" rpy="0 0 1.57"/>
 </joint>
-<joint name="Rigid1" type="fixed">
-  <origin xyz="0.029369 -0.014322 0.048" rpy="0 0 0"/>
+<joint name="lidar_joint" type="fixed">
   <parent link="base_link"/>
-  <child link="lidar_link"/>
+  <child link="laser"/>
+  <!--origin xyz="0 -0.03 0.15" rpy="0 0 1.57"/-->
+  <origin xyz="0 0 0.1" rpy="0 0 1.57"/>
 </joint>
-<joint name="Rigid2" type="fixed">
-  <origin xyz="0.029369 -0.014322 0.048" rpy="0 0 0"/>
-  <parent link="base_link"/>
-  <child link="lidar_1"/>
-</joint>
-<!--wheel joint-->
+<!--base-wheel joint-->
 <joint name="Rev3" type="continuous">
   <origin xyz="0.0 0.11454 0.02425" rpy="0 0 0"/>

Commit message: update

File: urdf_description/urdf/urdf.xacro (robot description, xacro)
@@ -4,4 +4,7 @@
 <xacro:include filename="$(find urdf_description)/urdf/urdf.trans" />
 <xacro:include filename="$(find urdf_description)/urdf/urdf.gazebo" />
+<link name="base_footprint">
+  <origin xyz="0 0 0" rpy="0 0 0"/>
+  </link>
 <link name="base_link">
   <!--inertial>
@@ -121,9 +124,13 @@
   <origin xyz="0 0 0.1" rpy="0 0 1.57"/>
 </joint>
-<joint name="lidar_joint" type="fixed">
+<joint name="dummy_joint" type="fixed">
+  <parent link="base_footprint"/>
+  <child link="base_link"/>
+  <origin xyz="0 0 0.048" rpy="0 0 1.57"/>
+</joint>
+<joint name="Rigid1" type="fixed">
+  <origin xyz="0.029369 -0.014322 0.048" rpy="0 0 0"/>
   <parent link="base_link"/>
-  <child link="laser"/>
-  <!--origin xyz="0 -0.03 0.15" rpy="0 0 1.57"/-->
-  <origin xyz="0 0 0.1" rpy="0 0 1.57"/>
+  <child link="lidar_link"/>
 </joint>
 <!--base-wheel joint-->

Commit message: update

File: urdf_description/urdf/urdf.xacro (robot description, xacro)
@@ -117,4 +117,10 @@
     </inertial>
 </link>
+<!--base-footprint joint-->
+<joint name="dummy_joint" type="fixed">
+  <parent link="base_footprint"/>
+  <child link="base_link"/>
+  <origin xyz="0 0 0" rpy="0 0 1.57"/>
+</joint>
 <!--base-lidar joint-->
 <joint name="lidar_joint" type="fixed">
@@ -123,9 +129,4 @@
   <!--origin xyz="0 -0.03 0.15" rpy="0 0 1.57"/-->
   <origin xyz="0 0 0.1" rpy="0 0 1.57"/>
-</joint>
-<joint name="dummy_joint" type="fixed">
-  <parent link="base_footprint"/>
-  <child link="base_link"/>
-  <origin xyz="0 0 0.048" rpy="0 0 1.57"/>
 </joint>
 <joint name="Rigid1" type="fixed">

Commit message: update

File: urdf_description/urdf/urdf.xacro (robot description, xacro)
@@ -125,5 +125,5 @@
   <child link="laser"/>
   <!--origin xyz="0 -0.03 0.15" rpy="0 0 1.57"/-->
-  <origin xyz="0 0 0.1" rpy="0 0 0"/>
+  <origin xyz="0.03 0 0.156" rpy="0 0 0"/>
 </joint>
 <joint name="Rigid1" type="fixed">

Commit message: update

File: urdf_description/urdf/urdf.xacro (robot description, xacro)
@@ -150,3 +150,73 @@
   <axis xyz="0.5 0.866025 -0.0"/>
 </joint>
+<xacro:property name="body_color" value="Gazebo/Black" />
+<xacro:property name="body_color1" value="Gazebo/Silver" />
+<xacro:property name="body_color2" value="Gazebo/Yellow" />
+<gazebo reference="base_link">
+  <material>${body_color1}</material>
+  <mu1>0.2</mu1>
+  <mu2>0.2</mu2>
+  <selfCollide>true</selfCollide>
+  <gravity>true</gravity>
+</gazebo>
+<gazebo reference="laser">
+  <material>${body_color2}</material>
+        <sensor name="laser" type="ray">
+            <pose> 0 0 0 0 0 0 </pose>
+            <visualize>true</visualize>
+            <update_rate>10</update_rate>
+            <ray>
+                <scan>
+                    <horizontal>
+                        <samples>360</samples>
+                        <min_angle>-3.14</min_angle>
+                        <max_angle>3.14</max_angle>
+                    </horizontal>
+                </scan>
+                <range>
+                    <min>0.15</min>
+                    <max>6</max>
+                </range>
+            </ray>
+            <plugin name="laser_controller" filename="libgazebo_ros_ray_sensor.so">
+                <ros>
+                    <argument>~/out:=scan</argument>
+                </ros>
+                <output_type>sensor_msgs/LaserScan</output_type>
+                <frame_name>laser_frame</frame_name>
+            </plugin>
+        </sensor>
+  <mu1>0.2</mu1>
+  <mu2>0.2</mu2>
+  <selfCollide>true</selfCollide>
+  <gravity>true</gravity>
+</gazebo>
+<gazebo reference="wheel_link_1">
+  <material>${body_color}</material>
+  <mu1>0.2</mu1>
+  <mu2>0.2</mu2>
+  <selfCollide>true</selfCollide>
+</gazebo>
+<gazebo reference="wheel_link_2">
+  <material>${body_color}</material>
+  <mu1>0.2</mu1>
+  <mu2>0.2</mu2>
+  <selfCollide>true</selfCollide>
+</gazebo>
+<gazebo reference="wheel_link_3">
+  <material>${body_color}</material>
+  <mu1>0.2</mu1>
+  <mu2>0.2</mu2>
+  <selfCollide>true</selfCollide>
+</gazebo>
+<gazebo>
+    <plugin name="object_controller" filename="libgazebo_ros_planar_move.so">
+      <commandTopic>joystickvelocity</commandTopic>
+      <odometryTopic>odom</odometryTopic>
+      <odometryFrame>odom</odometryFrame>
+      <odometryRate>20.0</odometryRate>
+      <robotBaseFrame>base_footprint</robotBaseFrame>
+      <publishTF>false</publishTF>
+    </plugin>
+</gazebo>
 </robot>

Commit message: roscd

File: urdf_description/urdf/urdf.xacro (robot description, xacro)
@@ -193,5 +193,5 @@
 </gazebo>
 <gazebo reference="wheel_link_1">
-  <material>${body_color}</material>
+  <material>${body_color1}</material>
   <mu1>0.2</mu1>
   <mu2>0.2</mu2>
@@ -199,5 +199,5 @@
 </gazebo>
 <gazebo reference="wheel_link_2">
-  <material>${body_color}</material>
+  <material>${body_color1}</material>
   <mu1>0.2</mu1>
   <mu2>0.2</mu2>
@@ -205,5 +205,5 @@
 </gazebo>
 <gazebo reference="wheel_link_3">
-  <material>${body_color}</material>
+  <material>${body_color1}</material>
   <mu1>0.2</mu1>
   <mu2>0.2</mu2>

Commit message: update

File: urdf_description/urdf/urdf.xacro (robot description, xacro)
@@ -160,5 +160,37 @@
   <gravity>true</gravity>
 </gazebo>
-<gazebo reference="laser">
+ <gazebo reference="laser">
+    <material>${body_color2}</material>
+    <sensor type="ray" name="lds_lfcd_sensor">
+      <pose>0 0 0 0 0 0</pose>
+      <visualize>true</visualize>
+      <update_rate>5</update_rate>
+      <ray>
+        <scan>
+          <horizontal>
+            <samples>360</samples>
+            <resolution>1</resolution>
+              <min_angle>-3.12413</min_angle>
+              <max_angle>3.14159</max_angle>
+          </horizontal>
+        </scan>
+        <range>
+          <min>0.120</min>
+          <max>10</max>
+          <resolution>0.01</resolution>
+        </range>
+        <noise>
+          <type>gaussian</type>
+          <mean>0.0</mean>
+          <stddev>0.01</stddev>
+        </noise>
+      </ray>
+      <plugin name="gazebo_ros_lds_lfcd_controller" filename="libgazebo_ros_laser.so">
+        <topicName>scan</topicName>
+        <frameName>laser</frameName>
+      </plugin>
+    </sensor>
+ </gazebo>
+<!--gazebo reference="laser">
   <material>${body_color2}</material>
         <sensor name="laser" type="ray">
@@ -191,5 +223,5 @@
   <selfCollide>true</selfCollide>
   <gravity>true</gravity>
-</gazebo>
+</gazebo!-->
 <gazebo reference="wheel_link_1">
   <material>${body_color1}</material>
@@ -212,5 +244,5 @@
 <gazebo>
     <plugin name="object_controller" filename="libgazebo_ros_planar_move.so">
-      <commandTopic>joystickvelocity</commandTopic>
+      <commandTopic>cmd_vel</commandTopic>
       <odometryTopic>odom</odometryTopic>
       <odometryFrame>odom</odometryFrame>

Commit message: update

File: urdf_description/urdf/urdf.xacro (robot description, xacro)
@@ -154,5 +154,5 @@
 <xacro:property name="body_color2" value="Gazebo/Yellow" />
 <gazebo reference="base_link">
-  <material>${body_color1}</material>
+  <material>${body_color2}</material>
   <mu1>0.2</mu1>
   <mu2>0.2</mu2>
@@ -171,5 +171,5 @@
             <samples>360</samples>
             <resolution>1</resolution>
-              <min_angle>-3.12413</min_angle>
+              <min_angle>-3.14159</min_angle>
               <max_angle>3.14159</max_angle>
           </horizontal>
@@ -192,36 +192,4 @@
     </sensor>
  </gazebo>
-<!--gazebo reference="laser">
-  <material>${body_color2}</material>
-        <sensor name="laser" type="ray">
-            <pose> 0 0 0 0 0 0 </pose>
-            <visualize>true</visualize>
-            <update_rate>40</update_rate>
-            <ray>
-                <scan>
-                    <horizontal>
-                        <samples>720</samples>
-                        <resolution>1</resolution>
-                        <min_angle>-3.12413</min_angle>
-                        <max_angle>3.14159</max_angle>
-                    </horizontal>
-                </scan>
-                <range>
-                    <min>0.15</min>
-                    <max>12</max>
-                    <resolution>0.01</resolution>
-                </range>
-            </ray>
-            <plugin name="laser_back" filename="libgazebo_ros_laser.so">
-                <output_type>sensor_msgs/LaserScan</output_type>
-                <frame_name>laser</frame_name>
-                <topicName>scan</topicName>
-            </plugin>
-        </sensor>
-  <mu1>0.2</mu1>
-  <mu2>0.2</mu2>
-  <selfCollide>true</selfCollide>
-  <gravity>true</gravity>
-</gazebo!-->
 <gazebo reference="wheel_link_1">
   <material>${body_color1}</material>

Commit message: joystick control multiple robot in gazebo

File: urdf_description/urdf/urdf.xacro (robot description, xacro)
@@ -154,5 +154,5 @@
 <xacro:property name="body_color2" value="Gazebo/Yellow" />
 <gazebo reference="base_link">
-  <material>${body_color2}</material>
+  <material>${body_color}</material>
   <mu1>0.2</mu1>
   <mu2>0.2</mu2>
@@ -164,5 +164,5 @@
     <sensor type="ray" name="lds_lfcd_sensor">
       <pose>0 0 0 0 0 0</pose>
-      <visualize>true</visualize>
+      <visualize>false</visualize>
       <update_rate>30</update_rate>
       <ray>

Commit message: xc continuous joint fixed, publish map odom static

File: urdf_description/urdf/urdf.xacro (robot description, xacro)
@@ -132,5 +132,6 @@
   <child link="lidar_link"/>
 </joint>
-<joint name="Rev3" type="continuous">
+<!--joint name="Rev3" type="continuous"-->
+<joint name="Rev3" type="fixed">
   <origin xyz="-0.103583 -0.006625 0.024" rpy="0 0 0"/>
   <parent link="base_link"/>
@@ -138,5 +139,5 @@
   <axis xyz="-1.0 -0.0 -0.0"/>
 </joint>
-<joint name="Rev4" type="continuous">
+<joint name="Rev4" type="fixed">
   <origin xyz="0.068227 -0.105819 0.024" rpy="0 0 0"/>
   <parent link="base_link"/>
@@ -144,5 +145,5 @@
   <axis xyz="0.5 -0.866025 -0.0"/>
 </joint>
-<joint name="Rev5" type="continuous">
+<joint name="Rev5" type="fixed">
   <origin xyz="0.068227 0.09257 0.024" rpy="0 0 0"/>
   <parent link="base_link"/>
