Commit message: spawn multi robot in map done

File: urdf_description/urdf/urdf.xacro (robot description, xacro)
@@ -155,5 +155,5 @@
 <xacro:property name="body_color2" value="Gazebo/Yellow" />
 <gazebo reference="base_link">
-  <material>${body_color}</material>
+  <material>${body_color1}</material>
   <mu1>0.2</mu1>
   <mu2>0.2</mu2>
@@ -162,5 +162,5 @@
 </gazebo>
  <gazebo reference="laser">
-    <material>${body_color2}</material>
+    <material>${body_color}</material>
     <sensor type="ray" name="lds_lfcd_sensor">
       <pose>0 0 0 0 0 0</pose>
@@ -193,4 +193,10 @@
     </sensor>
  </gazebo>
+<gazebo reference="lidar_link">
+  <material>${body_color}</material>
+  <mu1>0.2</mu1>
+  <mu2>0.2</mu2>
+  <selfCollide>true</selfCollide>
+</gazebo>
 <gazebo reference="wheel_link_1">
   <material>${body_color1}</material>

Commit message: add ensure goal pos but still slow

File: urdf_description/urdf/urdf.xacro (robot description, xacro)
@@ -30,5 +30,5 @@
   <inertial>
     <origin xyz="0.007650926996154439 -6.583497840632717e-05 7.082305684349283e-05" rpy="0 0 0"/>
-    <mass value="0.17051038938064"/>
+    <mass value="10.17051038938064"/>
     <inertia ixx="5e-05" iyy="3.2e-05" izz="3.2e-05" ixy="-0.0" iyz="-0.0" ixz="-0.0"/>
   </inertial>
@@ -50,5 +50,5 @@
   <inertial>
     <origin xyz="-0.0039033081055799 0.006580816821685306 3.642650617940307e-05" rpy="0 0 0"/>
-    <mass value="0.17051038938064"/>
+    <mass value="10.17051038938064"/>
     <inertia ixx="3.7e-05" iyy="4.6e-05" izz="3.2e-05" ixy="-8e-06" iyz="0.0" ixz="-0.0"/>
   </inertial>
@@ -70,5 +70,5 @@
   <inertial>
     <origin xyz="-0.0037745189185399014 -0.006655427439052869 7.703379049328954e-05" rpy="0 0 0"/>
-    <mass value="0.17051038938064"/>
+    <mass value="10.17051038938064"/>
     <inertia ixx="3.7e-05" iyy="4.6e-05" izz="3.2e-05" ixy="8e-06" iyz="-0.0" ixz="-0.0"/>
   </inertial>
@@ -201,18 +201,18 @@
 <gazebo reference="wheel_link_1">
   <material>${body_color1}</material>
-  <mu1>0.6</mu1>
-  <mu2>0.6</mu2>
+  <mu1>0.5</mu1>
+  <mu2>0.5</mu2>
   <selfCollide>true</selfCollide>
 </gazebo>
 <gazebo reference="wheel_link_2">
   <material>${body_color1}</material>
-  <mu1>0.6</mu1>
-  <mu2>0.6</mu2>
+  <mu1>0.5</mu1>
+  <mu2>0.5</mu2>
   <selfCollide>true</selfCollide>
 </gazebo>
 <gazebo reference="wheel_link_3">
   <material>${body_color1}</material>
-  <mu1>0.6</mu1>
-  <mu2>0.6</mu2>
+  <mu1>0.5</mu1>
+  <mu2>0.5</mu2>
   <selfCollide>true</selfCollide>
 </gazebo>

Commit message: done with ensurepath

File: urdf_description/urdf/urdf.xacro (robot description, xacro)
@@ -154,6 +154,8 @@
 <xacro:property name="body_color1" value="Gazebo/Silver" />
 <xacro:property name="body_color2" value="Gazebo/Yellow" />
+<xacro:property name="body_color3" value="Gazebo/Gray" />
+<xacro:property name="body_color4" value="Gazebo/White" />
 <gazebo reference="base_link">
-  <material>${body_color1}</material>
+  <material>${body_color4}</material>
   <mu1>0.2</mu1>
   <mu2>0.2</mu2>
@@ -200,5 +202,5 @@
 </gazebo>
 <gazebo reference="wheel_link_1">
-  <material>${body_color1}</material>
+  <material>${body_color3}</material>
   <mu1>0.5</mu1>
   <mu2>0.5</mu2>
@@ -206,5 +208,5 @@
 </gazebo>
 <gazebo reference="wheel_link_2">
-  <material>${body_color1}</material>
+  <material>${body_color3}</material>
   <mu1>0.5</mu1>
   <mu2>0.5</mu2>
@@ -212,5 +214,5 @@
 </gazebo>
 <gazebo reference="wheel_link_3">
-  <material>${body_color1}</material>
+  <material>${body_color3}</material>
   <mu1>0.5</mu1>
   <mu2>0.5</mu2>
